File: FCHardware/FCHardware.kicad_pcb (KiCad board)
At the start: 2 copper layers, 39 x 39 mm, 51 parts, among them J2 JST-4pin, J3 JST-8pin, J4 UJ20-C-H-G-SMT-2A-P16-TR, U1 ICM-42688-P, U2 STM32F405RGTx, U3 USBLC6-2SC6, U4 AP2112K-3.3, U5 TPSM63603

Commit message: Added silkscreen components naming
Parts:
- J2 RCV: renamed from J2
- J3 ESC: renamed from J3
- renumbered TP5 to TP3V3, TP4 to TP5V, TP1 to TPBoot, TP3 to TPGND, TP2 to TPReset
Other:
- board text added: "IMU"
- board text added: "LDO"
- board text added: "MCU"
Changed lines of the file:
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@@
 		(tags "inductor handsolder")
 		(property "Reference" "FB1"
-			(at 0 -1.65 0)
+			(at -3.1 0.1 0)
 			(layer "F.SilkS")
 			(effects
@@
 		(tags "capacitor handsolder")
 		(property "Reference" "C6"
-			(at 0 -1.43 90)
+			(at 2.2 0 180)
 			(layer "F.SilkS")
 			(effects
@@
 		(tags "resistor handsolder")
 		(property "Reference" "R8"
-			(at 0 -1.43 90)
+			(at -0.7 1.5 90)
 			(layer "F.SilkS")
 			(effects
@@
 		(descr "wire loop with bead as test point, loop diameter 1.8mm, hole diameter 1.0mm")
 		(tags "test point wire loop bead")
-		(property "Reference" "TP1"
+		(property "Reference" "TPBoot"
 			(at 0.7 2.5 0)
 			(layer "F.SilkS")
@@
 		(tags "capacitor handsolder")
 		(property "Reference" "C14"
-			(at 0 -1.43 0)
+			(at -1.4 -0.7 0)
 			(layer "F.SilkS")
 			(effects
@@
 		(tags "capacitor handsolder")
 		(property "Reference" "C3"
-			(at 0 -1.43 0)
+			(at -2.7 0.1 0)
 			(layer "F.SilkS")
 			(effects
@@
 		(tags "capacitor handsolder")
 		(property "Reference" "C12"
-			(at 0 -1.43 90)
+			(at -2.1 -0.7 180)
 			(layer "F.SilkS")
 			(effects
@@
 		(tags "capacitor handsolder")
 		(property "Reference" "C15"
-			(at 0 -1.43 90)
+			(at 0.146267 -1.4 270)
 			(layer "F.SilkS")
 			(effects
@@
 		(tags "resistor handsolder")
 		(property "Reference" "R1"
-			(at 0 -1.43 90)
+			(at 2.2 0.6 180)
 			(layer "F.SilkS")
 			(effects
@@
 		(descr "wire loop with bead as test point, loop diameter 1.8mm, hole diameter 1.0mm")
 		(tags "test point wire loop bead")
-		(property "Reference" "TP5"
-			(at 0.7 2.5 0)
+		(property "Reference" "TP3V3"
+			(at 0.3 2.5 0)
 			(layer "F.SilkS")
 			(effects
@@
 		(tags "capacitor handsolder")
 		(property "Reference" "C7"
-			(at 0 -1.43 90)
+			(at 0 1.5 90)
 			(layer "F.SilkS")
 			(effects
@@
 		(tags "capacitor handsolder")
 		(property "Reference" "C13"
-			(at 0 -1.43 0)
+			(at -1.3 -1.3 0)
 			(layer "F.SilkS")
 			(effects
@@
 		(tags "capacitor handsolder")
 		(property "Reference" "C5"
-			(at 0 -1.43 0)
+			(at 2.7 -0.4 0)
 			(layer "F.SilkS")
 			(effects
@@
 		(descr "wire loop with bead as test point, loop diameter 1.8mm, hole diameter 1.0mm")
 		(tags "test point wire loop bead")
-		(property "Reference" "TP3"
-			(at 0.7 2.5 0)
+		(property "Reference" "TPGND"
+			(at 0.5 2.4 0)
 			(layer "F.SilkS")
 			(effects
@@
 		(tags "TSOT-23-5 Hand-soldering")
 		(property "Reference" "U4"
-			(at 0 -2.45 0)
+			(at 0.08 -2.9 0)
 			(layer "F.SilkS")
 			(effects
@@
 		(tags "capacitor handsolder")
 		(property "Reference" "C1"
-			(at 0 -1.68 90)
+			(at -2.5 0 0)
 			(layer "F.SilkS")
 			(effects
@@
 		(tags "resistor handsolder")
 		(property "Reference" "R4"
-			(at 0 -1.43 0)
+			(at 1.7 0.8 0)
 			(layer "F.SilkS")
 			(effects
@@
 		(tags "resistor handsolder")
 		(property "Reference" "R9"
-			(at 0 -1.43 90)
+			(at -0.7 -1.2 90)
 			(layer "F.SilkS")
 			(effects
@@
 		(tags "capacitor handsolder")
 		(property "Reference" "C4"
-			(at 0 -1.68 0)
+			(at 0 1.8 0)
 			(layer "F.SilkS")
 			(effects
@@
 		(at 86.3125 96.8)
 		(property "Reference" "U1"
-			(at -0.176 -2.0048 0)
+			(at 0.6875 -1.9 0)
 			(layer "F.SilkS")
 			(effects
@@
 		(tags "capacitor handsolder")
 		(property "Reference" "C8"
-			(at 0 -1.43 0)
+			(at 0 1.4 0)
 			(layer "F.SilkS")
 			(effects
@@
 		(descr "wire loop with bead as test point, loop diameter 1.8mm, hole diameter 1.0mm")
 		(tags "test point wire loop bead")
-		(property "Reference" "TP4"
-			(at 0.7 2.5 0)
+		(property "Reference" "TP5V"
+			(at -0.1 2.5 0)
 			(layer "F.SilkS")
 			(effects
@@
 		(descr "JST SH series connector, BM04B-SRSS-TB (http://www.jst-mfg.com/product/pdf/eng/eSH.pdf), generated with kicad-footprint-generator")
 		(tags "connector JST SH vertical")
-		(property "Reference" "J2"
+		(property "Reference" "J2 RCV"
 			(at 0 0.175 0)
 			(layer "F.SilkS")
@@
 		(descr "Molex CLIK-Mate series connector, 502386-0870 (http://www.molex.com/pdm_docs/sd/5023860270_sd.pdf), generated with kicad-footprint-generator")
 		(tags "connector Molex CLIK-Mate horizontal")
-		(property "Reference" "J3"
+		(property "Reference" "J3 ESC"
 			(at 0.05 -0.25 0)
 			(layer "F.SilkS")
@@
 		(tags "capacitor handsolder")
 		(property "Reference" "C11"
-			(at 0 -1.43 0)
+			(at 1.55 1.25 0)
 			(layer "F.SilkS")
 			(effects
@@
 		(tags "capacitor handsolder")
 		(property "Reference" "C10"
-			(at 0 -1.43 0)
+			(at 1.8 1.1 0)
 			(layer "F.SilkS")
 			(effects
@@
 		(tags "capacitor handsolder")
 		(property "Reference" "C16"
-			(at 0 -1.43 90)
+			(at 2.4 0 180)
 			(layer "F.SilkS")
 			(effects
@@
 		(descr "wire loop with bead as test point, loop diameter 1.8mm, hole diameter 1.0mm")
 		(tags "test point wire loop bead")
-		(property "Reference" "TP2"
-			(at 0.7 2.5 0)
+		(property "Reference" "TPReset"
+			(at 1.1 2.5 0)
 			(layer "F.SilkS")
 			(effects
@@
 		(at 102.1 113.4 180)
 		(property "Reference" "U5"
-			(at 0.725 4.635 0)
+			(at -0.9 4.1 0)
 			(layer "B.SilkS")
 			(effects
@@
 		(tags "capacitor handsolder")
 		(property "Reference" "C19"
-			(at 0 1.85 0)
+			(at 0 -1.9 0)
 			(layer "B.SilkS")
 			(effects
@@
 		(tags "resistor handsolder")
 		(property "Reference" "R7"
-			(at 0 1.43 0)
+			(at 0 -1.4 0)
 			(layer "B.SilkS")
 			(effects
@@
 		(tags "capacitor handsolder")
 		(property "Reference" "C18"
-			(at 0 1.43 0)
+			(at -2.4 2 90)
 			(layer "B.SilkS")
 			(effects
@@
 		(tags "capacitor handsolder")
 		(property "Reference" "C17"
-			(at 0 1.43 0)
+			(at 0 1.4 0)
 			(layer "B.SilkS")
 			(effects
@@
 		(layer "Edge.Cuts")
 	)
+	(gr_text "IMU"
+		(at 85.2 94.9 0)
+		(layer "F.SilkS")
+		(effects
+			(font
+				(size 0.48 0.48)
+				(thickness 0.12)
+			)
+		)
+	)
+	(gr_text "MCU"
+		(at 100.2 98.1 0)
+		(layer "F.SilkS")
+		(effects
+			(font
+				(size 1.575055 1.575055)
+				(thickness 0.15)
+			)
+		)
+	)
+	(gr_text "LDO"
+		(at 117.1 110.3 0)
+		(layer "F.SilkS")
+		(effects
+			(font
+				(size 1 1)
+				(thickness 0.15)
+			)
+		)
+	)
 	(segment

Commit message: Added Easter Eggs, fixed test points
Parts:
- added G***: LOGO, FCFootprints:ConvLogo, F.Cu at (93.6, 112.9)
- 3V3: renamed from TP3V3; footprint TestPoint:TestPoint_Loop_D1.80mm_Drill1.0mm_Beaded -> TestPoint:TestPoint_Pad_D1.5mm
- 5V: renamed from TP5V; footprint TestPoint:TestPoint_Loop_D1.80mm_Drill1.0mm_Beaded -> TestPoint:TestPoint_Pad_D1.5mm
- BOOT: renamed from TPBoot; footprint TestPoint:TestPoint_Loop_D1.80mm_Drill1.0mm_Beaded -> TestPoint:TestPoint_Pad_D1.5mm
- GND: renamed from TPGND; footprint TestPoint:TestPoint_Loop_D1.80mm_Drill1.0mm_Beaded -> TestPoint:TestPoint_Pad_1.5x1.5mm
- J2: renamed from J2 RCV
- J3: renamed from J3 ESC
- RST: renamed from TPReset; footprint TestPoint:TestPoint_Loop_D1.80mm_Drill1.0mm_Beaded -> TestPoint:TestPoint_Pad_D1.5mm
Other:
- board text added: "Fly Fast Land Hard Send It Anyway"
- board text added: "HERE BE HOT"
- board text added: "I'M TRYING"
- board text added: "If found, return with LiPo"
- board text added: "If you can read this, flip me over."
- board text added: "PLUG ME GENTLY"
- board text added: "SKILL REQUIRED"
- board text added: "SPIN ME RIGHT ROUND"
